Commit message: Added camera support

File: robots/descriptions/go2_description/urdf/go2_description.urdf (robot description, URDF)
Before this commit: robot go2_description, 29 links, 28 joints
Links:
- added link camera, mass 0.1; collision box size=0.03 0.05 0.04; visual box size=0.03 0.05 0.04
Joints:
- added joint camera_joint: type fixed, parent Head_lower, child camera, origin xyz=0.05 0 0 rpy=0 -1.5708 0, axis 0 0 0

File: robots/descriptions/go2_description/xacro/robot_VLP.xacro (robot description, xacro)
@@ -80,4 +80,56 @@
         </collision>
     </link>
+    <link name="camera_link">
+        <inertial>
+            <mass value="0.1"/>
+            <origin xyz="0 0 0" rpy="0 0 0"/>
+            <inertia ixx="0.0001" ixy="0" ixz="0" iyy="0.0001" iyz="0" izz="0.0001"/>
+        </inertial>
+        <visual>
+            <origin xyz="0 0 0" rpy="0 -1.5708 0"/>  <!-- Orientación hacia adelante -->
+            <geometry>
+                <box size="0.05 0.03 0.04"/>  <!-- Ancho, alto, profundidad -->
+            </geometry>
+            <material name="black"/>
+        </visual>
+        <collision>
+            <origin xyz="0 0 0" rpy="0 -1.5708 0"/>
+            <geometry>
+                <box size="0.05 0.03 0.04"/>
+            </geometry>
+        </collision>
+    </link>
+    <joint name="camera_joint" type="fixed">
+        <origin xyz="0.25 0 0.1" rpy="0 0 0"/>  <!-- Posición frente al torso -->
+        <parent link="trunk"/>
+        <child link="camera_link"/>
+    </joint>
+    <!-- Configuración de Gazebo -->
+    <gazebo reference="camera_link">
+        <material>Gazebo/Black</material>
+        <sensor type="camera" name="camera_sensor">
+            <update_rate>30</update_rate>
+            <camera name="main">
+                <horizontal_fov>1.0472</horizontal_fov>  <!-- 60° -->
+                <image>
+                    <width>640</width>
+                    <height>480</height>
+                    <format>R8G8B8</format>
+                </image>
+                <clip>
+                    <near>0.05</near>
+                    <far>100</far>
+                </clip>
+            </camera>
+            <plugin name="camera_controller" filename="libgazebo_ros_camera.so">
+                <alwaysOn>true</alwaysOn>
+                <updateRate>30</updateRate>
+                <cameraName>camera</cameraName>
+                <imageTopicName>image_raw</imageTopicName>
+                <cameraInfoTopicName>camera_info</cameraInfoTopicName>
+                <frameName>camera_link</frameName>
+            </plugin>
+        </sensor>
+    </gazebo>
     <!--
     <joint name="load_joint" type="fixed">

Commit message: Added gps support

File: robots/descriptions/go2_description/urdf/go2_description.urdf (robot description, URDF)
Before this commit: robot go2_description, 30 links, 29 joints
Links:
- removed link camera
Joints:
- removed joint camera_joint

File: robots/descriptions/go2_description/xacro/robot_VLP.xacro (robot description, xacro)
@@ -80,4 +80,49 @@
         </collision>
     </link>
+    <!-- ============= GPS ============= -->
+    <!-- Agregar el enlace GPS -->
+    <link name="gps_link">
+    <inertial>
+        <origin xyz="0 0 0" rpy="0 0 0"/>
+        <mass value="0.01"/>
+        <inertia ixx="1e-6" ixy="0" ixz="0" iyy="1e-6" iyz="0" izz="1e-6"/>
+    </inertial>
+    <visual>
+        <origin xyz="0 0 0" rpy="0 0 0"/>
+        <geometry>
+        <sphere radius="0.02"/>
+        </geometry>
+        <material name="black">
+        <color rgba="0.1 0.1 0.1 1"/>
+        </material>
+    </visual>
+    <collision>
+        <origin xyz="0 0 0" rpy="0 0 0"/>
+        <geometry>
+        <sphere radius="0.02"/>
+        </geometry>
+    </collision>
+    </link>
+    <!-- Agregar la unión fija para el GPS -->
+    <joint name="gps_joint" type="fixed">
+    <parent link="trunk"/>
+    <child link="gps_link"/>
+    <origin xyz="0 0 0" rpy="0 0 0"/>
+    </joint>
+    <!-- Configuración de Gazebo para GPS -->
+    <gazebo reference="gps_link">
+    <sensor name="my_gps" type="gps">
+    <!-- ensure the sensor is active (required) -->
+    <always_on>true</always_on>
+    <update_rate>30</update_rate>
+    <plugin name="gps" filename="libgazebo_ros_gps_sensor.so">
+        <ros>
+        <!-- publish to /gps/data -->
+        <namespace>/gps</namespace>
+        <remapping>~/out:=fix</remapping>
+        </ros>
+    </plugin>
+    </sensor>
+    </gazebo>
     <link name="camera_link">
         <inertial>
